Commit message: Restructure 'models' folder.

File: wandrian_run/models/hokuyo/urdf/hokuyo.urdf.xacro (robot description, xacro)
@@ -1,21 +1,22 @@
 <?xml version="1.0" ?>
-<robot name="sensor_hokuyo" xmlns:xacro="http://ros.org/wiki/xacro">
+<robot name="model_hokuyo" xmlns:xacro="http://ros.org/wiki/xacro">
+  <xacro:include filename="$(find wandrian_run)/models/hokuyo/urdf/hokuyo_gazebo.urdf.xacro"/>
   <!-- Hokuyo 2D LIDAR -->
-  <xacro:macro name="sensor_hokuyo" params="parent">
+  <xacro:macro name="model_hokuyo" params="parent">
     <joint name="laser_sensor_joint" type="fixed">
-      <origin xyz="0.0 0.0 0.12" rpy="0.0 0.0 0.0" />
-      <parent link="base_link" />
-      <child link="laser_sensor_link" />
+      <origin xyz="0.0 0.0 0.15" rpy="0.0 0.0 0.0"/>
+      <parent link="${parent}"/>
+      <child link="laser_sensor_link"/>
     </joint>
     <link name="laser_sensor_link">
       <visual name="visual">
         <geometry>
-          <mesh filename="package://wandrian_run/models/hokuyo/meshes/hokuyo.dae" />
+          <mesh filename="package://wandrian_run/models/hokuyo/meshes/hokuyo.dae"/>
         </geometry>
       </visual>
       <inertial>
-        <mass value="0.000001" />
-        <origin xyz="0 0 0" />
-        <inertia ixx="0.0001" ixy="0.0" ixz="0.0" iyy="0.0001" iyz="0.0" izz="0.0001" />
+        <mass value="0.000001"/>
+        <origin xyz="0 0 0"/>
+        <inertia ixx="0.0001" ixy="0.0" ixz="0.0" iyy="0.0001" iyz="0.0" izz="0.0001"/>
       </inertial>
       <collision name="collision-base">
@@ -28,32 +29,10 @@
         <pose>0 0 0.0205 0 0 0</pose>
         <geometry>
-          <cylinder radius="0.021" length="0.029" />
+          <cylinder radius="0.021" length="0.029"/>
         </geometry>
       </collision>
-      <sensor name="laser" type="ray">
-        <pose>0.01 0 0.0175 0 -0 0</pose>
-        <ray>
-          <scan>
-            <horizontal>
-              <samples>640</samples>
-              <resolution>1</resolution>
-              <min_angle>-2.26889</min_angle>
-              <max_angle>2.268899</max_angle>
-            </horizontal>
-          </scan>
-          <range>
-            <min>0.08</min>
-            <max>10</max>
-            <resolution>0.01</resolution>
-          </range>
-        </ray>
-        <plugin name="laser" filename="libRayPlugin.so" />
-        <always_on>1</always_on>
-        <update_rate>30</update_rate>
-        <visualize>true</visualize>
-      </sensor>
     </link>
-    <!-- Set up laser gazebo details -->
-    <hokuyo_laser />
+    <!-- Set up Hokuyo Gazebo simulation details -->
+    <gazebo_hokuyo/>
   </xacro:macro>
 </robot>

File: wandrian_run/models/kobuki/urdf/kobuki.urdf.xacro (robot description, xacro)
@@ -1,12 +1,7 @@
 <?xml version="1.0" ?>
-<!--
-  This is not a standalone urdf for kobuki. It simply defines the 'kobuki' tag that can
-  be incorporated by other urdf files (e.g. turtlebot).
- -->
-<robot name="kobuki" xmlns:xacro="http://ros.org/wiki/xacro">
-  <xacro:include filename="$(find wandrian_run)/models/kobuki/urdf/common_properties.urdf.xacro"/>
+<robot name="model_kobuki" xmlns:xacro="http://ros.org/wiki/xacro">
   <xacro:include filename="$(find wandrian_run)/models/kobuki/urdf/kobuki_gazebo.urdf.xacro"/>
   <!-- Kobuki -->
-  <xacro:macro name="kobuki">
+  <xacro:macro name="model_kobuki">
     <link name="base_footprint"/>
     <!--
@@ -20,7 +15,7 @@
       -->
     <joint name="base_joint" type="fixed">
-      <origin xyz="0 0 0.0102" rpy="0 0 0" />
+      <origin xyz="0 0 0.0102" rpy="0 0 0"/>
       <parent link="base_footprint"/>
-      <child link="base_link" />
+      <child link="base_link"/>
     </joint>
     <link name="base_link">
@@ -28,5 +23,5 @@
         <geometry>
           <!-- new mesh -->
-          <mesh filename="package://wandrian_run/models/kobuki/meshes/main_body.dae" />
+          <mesh filename="package://wandrian_run/models/kobuki/meshes/main_body.dae"/>
         </geometry>
         <origin xyz="0.001 0 0.05199" rpy="0 0 0"/>
@@ -51,5 +46,5 @@
         <inertia ixx="0.019995" ixy="0.0" ixz="0.0"
                  iyy="0.019995" iyz="0.0"
-                 izz="0.03675" />
+                 izz="0.03675"/>
       </inertial>
     </link>
@@ -74,9 +69,9 @@
       </collision>
       <inertial>
-        <mass value="0.01" />
-        <origin xyz="0 0 0" />
-        <inertia ixx="0.001" ixy="0.0" ixz="0.0"
-                 iyy="0.001" iyz="0.0"
-                 izz="0.001" />
+        <mass value="0.01"/>
+        <origin xyz="0 0 0"/>
+        <inertia ixx="0.001" ixy="0.0" ixz="0.0"
+                 iyy="0.001" iyz="0.0"
+                 izz="0.001"/>
       </inertial>
     </link>
@@ -101,9 +96,9 @@
       </collision>
       <inertial>
-        <mass value="0.01" />
-        <origin xyz="0 0 0" />
-        <inertia ixx="0.001" ixy="0.0" ixz="0.0"
-                 iyy="0.001" iyz="0.0"
-                 izz="0.001" />
+        <mass value="0.01"/>
+        <origin xyz="0 0 0"/>
+        <inertia ixx="0.001" ixy="0.0" ixz="0.0"
+                 iyy="0.001" iyz="0.0"
+                 izz="0.001"/>
       </inertial>
     </link>
@@ -121,9 +116,9 @@
       </collision>
       <inertial>
-        <mass value="0.01" />
-        <origin xyz="0 0 0" />
-        <inertia ixx="0.001" ixy="0.0" ixz="0.0"
-                 iyy="0.001" iyz="0.0"
-                 izz="0.001" />
+        <mass value="0.01"/>
+        <origin xyz="0 0 0"/>
+        <inertia ixx="0.001" ixy="0.0" ixz="0.0"
+                 iyy="0.001" iyz="0.0"
+                 izz="0.001"/>
       </inertial>
     </link>
@@ -141,9 +136,9 @@
       </collision>
       <inertial>
-        <mass value="0.01" />
-        <origin xyz="0 0 0" />
-        <inertia ixx="0.001" ixy="0.0" ixz="0.0"
-                 iyy="0.001" iyz="0.0"
-                 izz="0.001" />
+        <mass value="0.01"/>
+        <origin xyz="0 0 0"/>
+        <inertia ixx="0.001" ixy="0.0" ixz="0.0"
+                 iyy="0.001" iyz="0.0"
+                 izz="0.001"/>
       </inertial>
     </link>
@@ -165,49 +160,47 @@
     </link>
     <joint name="cliff_sensor_left_joint" type="fixed">
-      <origin xyz="0.08734 0.13601 0.0214" rpy="0 ${M_PI/2} 0" />
-      <parent link="base_link"/>
-      <child link="cliff_sensor_left_link" />
+      <origin xyz="0.08734 0.13601 0.0214" rpy="0 ${M_PI/2} 0"/>
+      <parent link="base_link"/>
+      <child link="cliff_sensor_left_link"/>
     </joint>
     <link name="cliff_sensor_left_link">
       <inertial>
-        <mass value="0.0001" />
-        <origin xyz="0 0 0" />
+        <mass value="0.0001"/>
+        <origin xyz="0 0 0"/>
         <inertia ixx="0.0001" ixy="0.0" ixz="0.0"
                  iyy="0.0001" iyz="0.0"
-                 izz="0.0001" />
+                 izz="0.0001"/>
       </inertial>
     </link>
     <joint name="cliff_sensor_right_joint" type="fixed">
-      <origin xyz="0.085 -0.13601 0.0214" rpy="0 ${M_PI/2} 0" />
-      <parent link="base_link"/>
-      <child link="cliff_sensor_right_link" />
+      <origin xyz="0.085 -0.13601 0.0214" rpy="0 ${M_PI/2} 0"/>
+      <parent link="base_link"/>
+      <child link="cliff_sensor_right_link"/>
     </joint>
     <link name="cliff_sensor_right_link">
       <inertial>
-        <mass value="0.0001" />
-        <origin xyz="0 0 0" />
+        <mass value="0.0001"/>
+        <origin xyz="0 0 0"/>
         <inertia ixx="0.0001" ixy="0.0" ixz="0.0"
                  iyy="0.0001" iyz="0.0"
-                 izz="0.0001" />
+                 izz="0.0001"/>
       </inertial>
     </link>
     <joint name="cliff_sensor_front_joint" type="fixed">
-      <origin xyz="0.156 0.00 0.0214" rpy="0 ${M_PI/2} 0" />
-      <parent link="base_link"/>
-      <child link="cliff_sensor_front_link" />
+      <origin xyz="0.156 0.00 0.0214" rpy="0 ${M_PI/2} 0"/>
+      <parent link="base_link"/>
+      <child link="cliff_sensor_front_link"/>
     </joint>
     <link name="cliff_sensor_front_link">
       <inertial>
-        <mass value="0.0001" />
-        <origin xyz="0 0 0" />
+        <mass value="0.0001"/>
+        <origin xyz="0 0 0"/>
         <inertia ixx="0.0001" ixy="0.0" ixz="0.0"
                  iyy="0.0001" iyz="0.0"
-                 izz="0.0001" />
-      </inertial>
-    </link>
-    <!-- Kobuki Gazebo simulation details -->
-    <kobuki_sim />
+                 izz="0.0001"/>
+      </inertial>
+    </link>
+    <!-- Set up Kobuki Gazebo simulation details -->
+    <gazebo_kobuki/>
   </xacro:macro>
-  <xacro:include filename="$(find wandrian_run)/models/hokuyo/urdf/hokuyo.urdf.xacro"/>
-  <sensor_hokuyo parent="base_link"/>
 </robot>

File: wandrian_run/models/kobuki/urdf/kobuki_gazebo.urdf.xacro (robot description, xacro)
@@ -1,5 +1,17 @@
 <?xml version="1.0"?>
-<robot name="kobuki_sim" xmlns:xacro="http://ros.org/wiki/xacro">
-  <xacro:macro name="kobuki_sim">
+<robot name="gazebo_kobuki" xmlns:xacro="http://ros.org/wiki/xacro">
+  <xacro:macro name="gazebo_kobuki">
+    <gazebo reference="base_link">
+      <mu1>0.3</mu1>
+      <mu2>0.3</mu2>
+      <sensor type="contact" name="bumpers">
+        <always_on>1</always_on>
+        <update_rate>50.0</update_rate>
+        <visualize>true</visualize>
+        <contact>
+          <collision>base_footprint_collision_base_link</collision>
+        </contact>
+      </sensor>
+    </gazebo>
     <gazebo reference="wheel_left_link">
       <mu1>1.0</mu1>
@@ -34,106 +46,4 @@
       <maxVel>1.0</maxVel>
     </gazebo>
-    <gazebo reference="base_link">
-      <mu1>0.3</mu1>
-      <mu2>0.3</mu2>
-      <sensor type="contact" name="bumpers">
-        <always_on>1</always_on>
-        <update_rate>50.0</update_rate>
-        <visualize>true</visualize>
-        <contact>
-          <collision>base_footprint_collision_base_link</collision>
-        </contact>
-      </sensor>
-    </gazebo>
-    <gazebo reference="cliff_sensor_left_link">
-      <sensor type="ray" name="cliff_sensor_left">
-        <always_on>true</always_on>
-        <update_rate>50</update_rate>
-        <visualize>true</visualize>
-        <ray>
-          <scan>
-            <horizontal>
-              <samples>50</samples>
-              <resolution>1.0</resolution>
-              <min_angle>-0.0436</min_angle>  <!-- -2.5 degree -->
-              <max_angle>0.0436</max_angle> <!-- 2.5 degree -->
-            </horizontal>
-<!--            Can't use vertical rays until this bug is resolved: -->
-<!--            https://bitbucket.org/osrf/gazebo/issue/509/vertical-sensor-doesnt-works -->
-<!--             <vertical> -->
-<!--               <samples>50</samples> -->
-<!--               <resolution>1.0</resolution> -->
-<!--               <min_angle>-0.0436</min_angle>  -2.5 degree -->
-<!--               <max_angle>0.0436</max_angle> 2.5 degree -->
-<!--             </vertical> -->
-          </scan>
-          <range>
-            <min>0.01</min>
-            <max>0.15</max>
-            <resolution>1.0</resolution>
-          </range>
-        </ray>
-      </sensor>
-    </gazebo>
-    <gazebo reference="cliff_sensor_right_link">
-      <sensor type="ray" name="cliff_sensor_right">
-        <always_on>true</always_on>
-        <update_rate>50</update_rate>
-        <visualize>true</visualize>
-        <ray>
-          <scan>
-            <horizontal>
-              <samples>50</samples>
-              <resolution>1.0</resolution>
-              <min_angle>-0.0436</min_angle>  <!-- -2.5 degree -->
-              <max_angle>0.0436</max_angle> <!-- 2.5 degree -->
-            </horizontal>
-<!--            Can't use vertical rays until this bug is resolved: -->
-<!--            https://bitbucket.org/osrf/gazebo/issue/509/vertical-sensor-doesnt-works -->
-<!--             <vertical> -->
-<!--               <samples>50</samples> -->
-<!--               <resolution>1.0</resolution> -->
-<!--               <min_angle>-0.0436</min_angle>  -2.5 degree -->
-<!--               <max_angle>0.0436</max_angle> 2.5 degree -->
-<!--             </vertical> -->
-          </scan>
-          <range>
-            <min>0.01</min>
-            <max>0.15</max>
-            <resolution>1.0</resolution>
-          </range>
-        </ray>
-      </sensor>
-    </gazebo>
-    <gazebo reference="cliff_sensor_front_link">
-      <sensor type="ray" name="cliff_sensor_front">
-        <always_on>true</always_on>
-        <update_rate>50</update_rate>
-        <visualize>true</visualize>
-        <ray>
-          <scan>
-            <horizontal>
-              <samples>50</samples>
-              <resolution>1.0</resolution>
-              <min_angle>-0.0436</min_angle>  <!-- -2.5 degree -->
-              <max_angle>0.0436</max_angle> <!-- 2.5 degree -->
-            </horizontal>
-<!--             Can't use vertical rays until this bug is resolved: -->
-<!--            https://bitbucket.org/osrf/gazebo/issue/509/vertical-sensor-doesnt-works -->
-<!--             <vertical> -->
-<!--               <samples>50</samples> -->
-<!--               <resolution>1.0</resolution> -->
-<!--               <min_angle>-0.0436</min_angle>  -2.5 degree -->
-<!--               <max_angle>0.0436</max_angle> 2.5 degree -->
-<!--             </vertical> -->
-          </scan>
-          <range>
-            <min>0.01</min>
-            <max>0.15</max>
-            <resolution>1.0</resolution>
-          </range>
-        </ray>
-      </sensor>
-    </gazebo>
     <gazebo reference="gyro_link">
      <sensor type="imu" name="imu">
@@ -160,4 +70,94 @@
       </sensor>
     </gazebo>
+    <gazebo reference="cliff_sensor_left_link">
+      <sensor type="ray" name="cliff_sensor_left">
+        <always_on>true</always_on>
+        <update_rate>50</update_rate>
+        <visualize>true</visualize>
+        <ray>
+          <scan>
+            <horizontal>
+              <samples>50</samples>
+              <resolution>1.0</resolution>
+              <min_angle>-0.0436</min_angle>  <!-- -2.5 degree -->
+              <max_angle>0.0436</max_angle> <!-- 2.5 degree -->
+            </horizontal>
+            <!-- Can't use vertical rays until this bug is resolved: -->
+            <!-- https://bitbucket.org/osrf/gazebo/issue/509/vertical-sensor-doesnt-works -->
+            <!-- <vertical> -->
+              <!-- <samples>50</samples> -->
+              <!-- <resolution>1.0</resolution> -->
+              <!-- <min_angle>-0.0436</min_angle>  -2.5 degree -->
+              <!-- <max_angle>0.0436</max_angle> 2.5 degree -->
+            <!-- </vertical> -->
+          </scan>
+          <range>
+            <min>0.01</min>
+            <max>0.15</max>
+            <resolution>1.0</resolution>
+          </range>
+        </ray>
+      </sensor>
+    </gazebo>
+    <gazebo reference="cliff_sensor_right_link">
+      <sensor type="ray" name="cliff_sensor_right">
+        <always_on>true</always_on>
+        <update_rate>50</update_rate>
+        <visualize>true</visualize>
+        <ray>
+          <scan>
+            <horizontal>
+              <samples>50</samples>
+              <resolution>1.0</resolution>
+              <min_angle>-0.0436</min_angle>  <!-- -2.5 degree -->
+              <max_angle>0.0436</max_angle> <!-- 2.5 degree -->
+            </horizontal>
+            <!-- Can't use vertical rays until this bug is resolved: -->
+            <!-- https://bitbucket.org/osrf/gazebo/issue/509/vertical-sensor-doesnt-works -->
+            <!-- <vertical> -->
+              <!-- <samples>50</samples> -->
+              <!-- <resolution>1.0</resolution> -->
+              <!-- <min_angle>-0.0436</min_angle>  -2.5 degree -->
+              <!-- <max_angle>0.0436</max_angle> 2.5 degree -->
+            <!-- </vertical> -->
+          </scan>
+          <range>
+            <min>0.01</min>
+            <max>0.15</max>
+            <resolution>1.0</resolution>
+          </range>
+        </ray>
+      </sensor>
+    </gazebo>
+    <gazebo reference="cliff_sensor_front_link">
+      <sensor type="ray" name="cliff_sensor_front">
+        <always_on>true</always_on>
+        <update_rate>50</update_rate>
+        <visualize>true</visualize>
+        <ray>
+          <scan>
+            <horizontal>
+              <samples>50</samples>
+              <resolution>1.0</resolution>
+              <min_angle>-0.0436</min_angle>  <!-- -2.5 degree -->
+              <max_angle>0.0436</max_angle> <!-- 2.5 degree -->
+            </horizontal>
+            <!-- Can't use vertical rays until this bug is resolved: -->
+            <!-- https://bitbucket.org/osrf/gazebo/issue/509/vertical-sensor-doesnt-works -->
+            <!-- <vertical> -->
+              <!-- <samples>50</samples> -->
+              <!-- <resolution>1.0</resolution> -->
+              <!-- <min_angle>-0.0436</min_angle>  -2.5 degree -->
+              <!-- <max_angle>0.0436</max_angle> 2.5 degree -->
+            <!-- </vertical> -->
+          </scan>
+          <range>
+            <min>0.01</min>
+            <max>0.15</max>
+            <resolution>1.0</resolution>
+          </range>
+        </ray>
+      </sensor>
+    </gazebo>
     <gazebo>
       <plugin name="kobuki_controller" filename="libgazebo_ros_kobuki.so">
@@ -178,30 +178,3 @@
     </gazebo>
   </xacro:macro>
-  <!-- Hokuyo LIDAR for simulation -->
-  <xacro:macro name="hokuyo_laser">
-    <gazebo reference="laser_sensor_link">
-      <sensor name="laser" type="ray">
-        <pose>0.01 0 0.0175 0 0 0</pose>
-        <ray>
-          <scan>
-            <horizontal>
-              <samples>640</samples>
-              <resolution>1</resolution>
-              <min_angle>-1.57078</min_angle>
-              <max_angle>1.57078</max_angle>
-            </horizontal>
-          </scan>
-          <range>
-            <min>0.1</min>
-            <max>0.4</max>
-            <resolution>0.01</resolution>
-          </range>
-        </ray>
-        <plugin name="laser" filename="libRayPlugin.so" />
-        <always_on>1</always_on>
-        <update_rate>30</update_rate>
-        <visualize>true</visualize>
-      </sensor>
-    </gazebo>
-  </xacro:macro>
 </robot>

File: wandrian_run/models/robot/urdf/common_properties.urdf.xacro (robot description, xacro)
@@ -4,5 +4,5 @@
  -->
 <robot name="xacro_properties" xmlns:xacro="http://ros.org/wiki/xacro">
-  <xacro:property name="M_PI" value="3.1415926535897931" />
+  <xacro:property name="M_PI" value="3.1415926535897931"/>
   <xacro:property name="material_white">
     <material name="white">
